File: beer_ide_kicad/beer_ide_kicad.kicad_pcb (KiCad board)
At the start: 2 copper layers, 101.6 x 65.3 mm, 17 parts, among them CN1 MSX_SLOT_CON, J1 Sound IN, U1 8255A, U2 74LS32, U3 74LS30, U4 74LS04, U5 27128

Commit message: Add files via upload
Parts:
- U1: footprint Package_DIP:DIP-40_W15.24mm_Socket -> MSXmakers:DIP-40c_W15.24mm_LongPads
- U2, U3, U4: footprint Package_DIP:DIP-14_W7.62mm_Socket -> MSXmakers:DIP-14c_W7.62mm_LongPads
- U5: footprint Package_DIP:DIP-28_W15.24mm_Socket -> MSXmakers:DIP-28c_W15.24mm_Socket_LongPads
- moved U2 0.05 mm to (190.4, 60.9)
- moved U3 0.05 mm to (190.5, 76.2)
Routing:
- net /A2: track 67.7 -> 51.5 mm, vias 2 -> 0
- net GND: track 310.5 -> 308.6 mm
- net /RESET: track 51.3 -> 52.2 mm
- net /A9: track 23.0 -> 22.2 mm
- net /~{WR}: track 68.1 -> 67.4 mm
- net VCC: track 284.3 -> 284.9 mm
- net /~{RD}: track 79.7 -> 80.3 mm
- net /A5: track 88.3 -> 87.7 mm
- net /A6: track 63.2 -> 62.6 mm
Other:
- board text added: "MSX-BEER 202 v.1.2 Konami Case"
- board text added: "MSXmakers! 2023"
- board text removed: "MSX-BEER 202 v. 1.1 Konami Case"
- board text removed: "MSXmakers! 2021"
